File: pages/lowside_quad.kicad_sch (KiCad schematic)
At the start: 4 parts

Commit message: update
Other:
- company: ecu-TECH -> gerEFI
- title: ecu-TECH Proteus -> gerEFI Proteus
Changed lines of the file:
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@@
   (paper "A4")
   (title_block
-    (title "ecu-TECH Proteus")
+    (title "gerEFI Proteus")
     (date "2022-04-09")
     (rev "v0.7")
-    (company "ecu-TECH")
+    (company "gerEFI")
     (comment 1 "github.com/mck1117/proteus")
-    (comment 2 "ecu-tech.com/s/proteus")
+    (comment 2 "gerefi.com/s/proteus")
   )
   (junction (at 67.945 73.66) (diameter 0) (color 0 0 0 0)
